Commit message: Add conversion functions

File: module/actuation/Kinematics/data/nugus.urdf (robot description, URDF)
Before this commit: robot onshape, 23 links, 22 joints
Joints:
- joint right_ankle_pitch: axis 0 0 1 -> 0 0 -1

Commit message: Update SensorFilter kinematics

File: module/actuation/Kinematics/data/nugus.urdf (robot description, URDF)
Before this commit: robot onshape, 23 links, 22 joints
Joints:
- removed joint left_shoulder_yaw
- removed joint right_shoulder_yaw
- added joint left_shoulder_roll: type revolute, parent left_shoulder, child left_upper_arm, origin xyz=-0.0100012 0 -0.0479124 rpy=1.5708 -1.93145e-15 -3.14159, axis 0 0 1, limit lower=-3.14159 upper=3.14159 effort=1.5 velocity=22
- added joint right_shoulder_roll: type revolute, parent right_shoulder, child right_upper_arm, origin xyz=-0.0100012 2.77556e-17 -0.0479124 rpy=-1.5708 -3.12007e-15 3.14159, axis 0 0 1, limit lower=-3.14159 upper=3.14159 effort=1.5 velocity=22

Commit message: Add left and right camera [WIP]

File: module/actuation/Kinematics/data/nugus.urdf (robot description, URDF)
Before this commit: robot onshape, 23 links, 22 joints
Links:
- added link left_camera, mass 0; collision mesh filename=left_camera_collision.stl; visual mesh filename=left_camera_visual.stl
- added link right_camera, mass 0; collision mesh filename=right_camera_collision.stl; visual mesh filename=right_camera_visual.stl
- link left_upper_leg: mass 0.164996 -> 0.136613
- link right_upper_leg: mass 0.164996 -> 0.136613
Joints:
- removed joint left_knee_pitch
- removed joint right_knee_pitch
- added joint left_camera: type fixed, parent head, child left_camera, origin xyz=0.0648803 0.0699522 0.033795 rpy=1.5708 7.65706e-15 1.6057, axis 0 0 1, limit effort=1 velocity=20
- added joint left_knee: type revolute, parent left_upper_leg, child left_lower_leg, origin xyz=0.206046 -0.0569501 1.51268e-15 rpy=-3.14159 1.05543e-15 -4.06897e-14, axis 0 0 -1, limit lower=-3.14159 upper=3.14159 effort=1 velocity=20
- added joint right_camera: type fixed, parent head, child right_camera, origin xyz=0.0648803 0.0699522 -0.034205 rpy=1.5708 7.65265e-15 1.6057, axis 0 0 1, limit effort=1 velocity=20
- added joint right_knee: type revolute, parent right_upper_leg, child right_lower_leg, origin xyz=0.206046 -0.0569501 -1.66533e-16 rpy=1.79345e-17 -1.0453e-16 -1.11022e-16, axis 0 0 1, limit lower=-3.14159 upper=3.14159 effort=1 velocity=20
- joint left_ankle_pitch: axis 0 0 1 -> 0 0 -1; limit lower=-3.14159 upper=3.14159 effort=1.5 velocity=22 -> lower=-3.14159 upper=3.14159 effort=1 velocity=20; origin xyz=0.200203 -3.25261e-17 2.27963e-09 rpy=4.2823e-15 8.25556e-15 1.5708 -> xyz=0.200203 -3.46945e-17 2.28591e-09 rpy=7.77156e-16 3.63979e-15 1.5708
- joint left_ankle_roll: limit lower=-3.14159 upper=3.14159 effort=1.5 velocity=22 -> lower=-3.14159 upper=3.14159 effort=1 velocity=20; origin xyz=4.34742e-09 4.58116e-10 -3.08702e-09 rpy=1.5708 3.11019e-14 -1.5708 -> xyz=4.34741e-09 4.48776e-10 -3.0933e-09 rpy=1.5708 -1.69309e-14 -1.5708
- joint left_elbow_pitch: limit lower=-3.14159 upper=3.14159 effort=1.5 velocity=22 -> lower=-3.14159 upper=3.14159 effort=1 velocity=20
- joint left_foot_base: limit effort=1.5 velocity=22 -> effort=1 velocity=20; origin xyz=0.0360246 2.77556e-17 1.30104e-18 rpy=8.86985e-31 -1.5708 0 -> xyz=0.0360246 1.38778e-17 1.38778e-17 rpy=1.96766e-30 -1.5708 0
- joint left_hip_pitch: limit lower=-3.14159 upper=3.14159 effort=1.5 velocity=22 -> lower=-3.14159 upper=3.14159 effort=1 velocity=20; origin xyz=0 1.38778e-17 6.93889e-18 rpy=-1.5708 -9.99201e-16 9.62078e-15 -> xyz=-6.93889e-18 6.93889e-18 1.04083e-17 rpy=1.5708 -9.99201e-16 9.62078e-15
- joint left_hip_roll: limit lower=-3.14159 upper=3.14159 effort=1.5 velocity=22 -> lower=-3.14159 upper=3.14159 effort=1 velocity=20; origin xyz=6.93889e-18 0.0221332 -0.0545 rpy=-1.5708 1.5708 0 -> xyz=0 0.0221332 -0.0545 rpy=-1.5708 1.5708 0
- joint left_hip_yaw: limit lower=-3.14159 upper=3.14159 effort=1.5 velocity=22 -> lower=-3.14159 upper=3.14159 effort=1 velocity=20
- joint left_shoulder_pitch: limit lower=-3.14159 upper=3.14159 effort=1.5 velocity=22 -> lower=-3.14159 upper=3.14159 effort=1 velocity=20
- joint left_shoulder_roll: limit lower=-3.14159 upper=3.14159 effort=1.5 velocity=22 -> lower=-3.14159 upper=3.14159 effort=1 velocity=20
- joint neck_pitch: limit lower=-3.14159 upper=3.14159 effort=1.5 velocity=22 -> lower=-3.14159 upper=3.14159 effort=1 velocity=20
- joint neck_yaw: limit lower=-3.14159 upper=3.14159 effort=1.5 velocity=22 -> lower=-3.14159 upper=3.14159 effort=1 velocity=20
- joint right_ankle_pitch: axis 0 0 -1 -> 0 0 1; limit lower=-3.14159 upper=3.14159 effort=1.5 velocity=22 -> effort=1 velocity=20; origin xyz=0.200203 3.29597e-17 2.27963e-09 rpy=3.14159 1.13004e-15 1.5708 -> xyz=0.200203 -3.46945e-17 0 rpy=-1.5432e-16 3.69866e-16 -1.5708
- joint right_ankle_roll: limit lower=-3.14159 upper=3.14159 effort=1.5 velocity=22 -> lower=-3.14159 upper=3.14159 effort=1 velocity=20; origin xyz=4.34741e-09 -4.58126e-10 3.08702e-09 rpy=-1.5708 -1.2536e-14 1.5708 -> xyz=4.34742e-09 -1.67644e-14 1.61479e-09 rpy=-1.5708 9.20375e-14 1.5708
- joint right_elbow_pitch: limit lower=-3.14159 upper=3.14159 effort=1.5 velocity=22 -> lower=-3.14159 upper=3.14159 effort=1 velocity=20
- joint right_foot_base: limit effort=1.5 velocity=22 -> effort=1 velocity=20; origin xyz=0.0360246 1.38778e-17 6.93889e-18 rpy=1.91535e-30 -1.5708 0 -> xyz=0.0360246 -6.93889e-18 6.93889e-18 rpy=-3.28467e-28 -1.5708 0
- joint right_hip_pitch: limit lower=-3.14159 upper=3.14159 effort=1.5 velocity=22 -> lower=-3.14159 upper=3.14159 effort=1 velocity=20; origin xyz=-2.08167e-17 -6.93889e-18 6.93889e-18 rpy=-1.5708 -3.91904e-27 -2.30022e-27 -> xyz=-1.38778e-17 6.93889e-18 6.93889e-18 rpy=1.5708 2.94117e-27 -9.49198e-31
- joint right_hip_roll: limit lower=-3.14159 upper=3.14159 effort=1.5 velocity=22 -> lower=-3.14159 upper=3.14159 effort=1 velocity=20; origin xyz=6.93889e-18 -0.0221332 -0.0545 rpy=1.5708 1.5708 0 -> xyz=0 -0.0221332 -0.0545 rpy=1.5708 1.5708 0
- joint right_hip_yaw: limit lower=-3.14159 upper=3.14159 effort=1.5 velocity=22 -> lower=-3.14159 upper=3.14159 effort=1 velocity=20
- joint right_shoulder_pitch: limit lower=-3.14159 upper=3.14159 effort=1.5 velocity=22 -> lower=-3.14159 upper=3.14159 effort=1 velocity=20
- joint right_shoulder_roll: limit lower=-3.14159 upper=3.14159 effort=1.5 velocity=22 -> lower=-3.14159 upper=3.14159 effort=1 velocity=20

Commit message: Update nugus.urdf

File: module/actuation/Kinematics/data/nugus.urdf (robot description, URDF)
Before this commit: robot onshape, 25 links, 24 joints
Links:
- link torso: mass 2.92465 -> 1.83264
Joints:
- joint left_ankle_pitch: axis 0 0 -1 -> 0 0 1; origin xyz=0.200203 -3.46945e-17 2.28591e-09 rpy=7.77156e-16 3.63979e-15 1.5708 -> xyz=0.200203 -3.46945e-17 6.93889e-18 rpy=-3.05311e-15 5.55112e-17 -2.87748e-14
- joint left_ankle_roll: origin xyz=4.34741e-09 4.48776e-10 -3.0933e-09 rpy=1.5708 -1.69309e-14 -1.5708 -> xyz=0 0 6.93889e-18 rpy=1.5708 3.37316e-16 -3.88578e-16
- joint left_camera: origin xyz=0.0648803 0.0699522 0.033795 rpy=1.5708 7.65706e-15 1.6057 -> xyz=-0.0648803 0.0699522 -0.033795 rpy=-1.5708 1.63801e-13 1.53589
- joint left_elbow_pitch: origin xyz=0.1575 5.57465e-05 -0.02695 rpy=1.5708 -7.49418e-30 -2.00673e-14 -> xyz=0.1575 -5.57465e-05 0.02695 rpy=1.5708 1.5708 0
- joint left_foot_base: origin xyz=0.0360246 1.38778e-17 1.38778e-17 rpy=1.96766e-30 -1.5708 0 -> xyz=0.0360247 0 6.93889e-18 rpy=-1.71429e-29 -1.5708 0
- joint left_hip_pitch: origin xyz=-6.93889e-18 6.93889e-18 1.04083e-17 rpy=1.5708 -9.99201e-16 9.62078e-15 -> xyz=0 -6.93889e-18 -1.38778e-17 rpy=-1.5708 -1.29896e-14 3.34849e-14
- joint left_hip_roll: origin xyz=0 0.0221332 -0.0545 rpy=-1.5708 1.5708 0 -> xyz=0.0221332 0 -0.0545 rpy=-4.55628e-30 1.5708 0
- joint left_hip_yaw: origin xyz=0 0.055 0 rpy=1.00616e-25 -1.69834e-26 -1.5708 -> xyz=7.63278e-17 0.055 0 rpy=-5.43064e-25 -3.21985e-24 6.16346e-16
- joint left_knee: axis 0 0 -1 -> 0 0 1; origin xyz=0.206046 -0.0569501 1.51268e-15 rpy=-3.14159 1.05543e-15 -4.06897e-14 -> xyz=0.206046 0.0569501 -1.44745e-14 rpy=-4.42146e-14 -3.94129e-15 -1.40554e-13
- joint left_shoulder_pitch: origin xyz=-2.0498e-17 0.077 0.17725 rpy=-1.5708 1.07261e-15 -3.14159 -> xyz=-5.659e-18 0.077 0.17725 rpy=1.5708 1.5708 0
- joint left_shoulder_roll: origin xyz=-0.0100012 0 -0.0479124 rpy=1.5708 -1.93145e-15 -3.14159 -> xyz=0 0.0100012 -0.0479124 rpy=-1.5708 -3.06087e-14 1.5708
- joint neck_pitch: origin xyz=-0.00024471 0.000255294 -0.0481 rpy=6.12323e-17 1.5708 0 -> xyz=-0.00024471 -0.000255294 0.0481 rpy=-1.5708 1.5708 0
- joint neck_yaw: origin xyz=-0.008 2.36302e-16 0.20825 rpy=3.14159 -2.77556e-16 1.5708 -> xyz=-0.008 2.09034e-16 0.20825 rpy=-1.1045e-15 2.10942e-15 -3.14159
- joint right_ankle_pitch: origin xyz=0.200203 -3.46945e-17 0 rpy=-1.5432e-16 3.69866e-16 -1.5708 -> xyz=0.200203 4.85723e-17 -6.93889e-18 rpy=1.88738e-15 -2.83277e-16 1.06524e-14
- joint right_ankle_roll: origin xyz=4.34742e-09 -1.67644e-14 1.61479e-09 rpy=-1.5708 9.20375e-14 1.5708 -> xyz=1.27676e-15 1.249e-16 -8.46545e-16 rpy=1.5708 -1.11022e-15 7.94382e-15
- joint right_camera: origin xyz=0.0648803 0.0699522 -0.034205 rpy=1.5708 7.65265e-15 1.6057 -> xyz=-0.0648803 0.0699522 0.034205 rpy=-1.5708 1.63801e-13 1.53589
- joint right_elbow_pitch: origin xyz=0.1575 -5.57465e-05 -0.02695 rpy=1.5708 4.09672e-14 -1.50852e-14 -> xyz=0.1575 5.57465e-05 0.02695 rpy=1.5708 1.5708 0
- joint right_foot_base: origin xyz=0.0360246 -6.93889e-18 6.93889e-18 rpy=-3.28467e-28 -1.5708 0 -> xyz=0.0360247 -1.38778e-17 0 rpy=-7.57306e-29 -1.5708 0
- joint right_hip_pitch: origin xyz=-1.38778e-17 6.93889e-18 6.93889e-18 rpy=1.5708 2.94117e-27 -9.49198e-31 -> xyz=-1.249e-16 0 3.81639e-17 rpy=-1.5708 -1.66533e-16 3.79139e-29
- joint right_hip_roll: origin xyz=0 -0.0221332 -0.0545 rpy=1.5708 1.5708 0 -> xyz=0.0221332 0 -0.0545 rpy=1.36238e-31 1.5708 0
- joint right_hip_yaw: origin xyz=-6.93889e-18 -0.055 -5.55112e-17 rpy=1.56194e-28 1.0176e-28 1.5708 -> xyz=-6.93889e-18 -0.055 -5.55112e-17 rpy=-1.44515e-26 2.05167e-26 2.3927e-15
- joint right_knee: origin xyz=0.206046 -0.0569501 -1.66533e-16 rpy=1.79345e-17 -1.0453e-16 -1.11022e-16 -> xyz=0.206046 0.0569501 -7.16788e-15 rpy=-7.0209e-15 3.9968e-14 -5.66214e-15
- joint right_shoulder_pitch: origin xyz=-3.8548e-17 -0.077 0.17725 rpy=1.5708 -5.87966e-17 -3.14159 -> xyz=-3.55526e-17 -0.077 0.17725 rpy=1.5708 1.5708 0
- joint right_shoulder_roll: origin xyz=-0.0100012 2.77556e-17 -0.0479124 rpy=-1.5708 -3.12007e-15 3.14159 -> xyz=0 0.0100012 0.0479124 rpy=-1.5708 4.32987e-15 1.5708

Commit message: Update nugus.urdf

File: module/actuation/Kinematics/data/nugus.urdf (robot description, URDF)
Before this commit: robot onshape, 25 links, 24 joints
Links:
- link head: geometry collision box size=0.16223767679184675 0.15564338862895966 0.1575121507048607; visual mesh filename=head_visual.stl
- link left_ankle: geometry collision box size=0.06627646926790476 0.09438799507915974 0.05529999919235706; visual mesh filename=left_ankle_visual.stl
- link left_camera: mass 0 -> 1.01635e-15; geometry collision box size=9.999999747378752e-06 1.0163475963054225e-05 9.999999747323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; visual mesh filename=left_camera_visual.stl
- link left_foot: geometry collision box size=0.05699313431978226 0.13158147037029266 0.21582108736038208; visual mesh filename=left_foot_visual.stl
- link left_foot_base: mass 0 -> 1.01635e-23; geometry collision box size=9.999999747378752e-06 1.0163475963054225e-05 9.999999747378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; visual mesh filename=left_foot_base_visual.stl
- link left_hip_roll: geometry collision box size=0.07245294097810984 0.05529999919235706 0.09385000355541706; visual mesh filename=left_hip_roll_visual.stl
- link left_hip_yaw: geometry collision box size=0.10850000381469727 0.09402551129460335 0.07350000609436158; visual mesh filename=left_hip_yaw_visual.stl
- link left_lower_arm: geometry collision box size=0.08257202059030533 0.25829844921827316 0.050877589732408524; visual mesh filename=left_lower_arm_visual.stl
- link left_lower_leg: geometry collision box size=0.2292028944939375 0.03099999949336052 0.07800000160932541; visual mesh filename=left_lower_leg_visual.stl
- link left_shoulder: geometry collision box size=0.07999999821186066 0.08144209161400795 0.0793731525540351; visual mesh filename=left_shoulder_visual.stl
- link left_upper_arm: mass 0.13422 -> 0.29923; geometry collision box size=0.22483809292316437 0.07902275025844574 0.08959516510367393; visual mesh filename=left_upper_arm_visual.stl
- link left_upper_leg: mass 0.136613 -> 0.313357; geometry collision box size=0.2462693639099598 0.09347053803503513 0.0729999989271164; visual mesh filename=left_upper_leg_visual.stl
- link neck: mass 0 -> 0.165011; geometry collision box size=0.04019999876618385 0.05000000074505806 0.062835298711434; visual mesh filename=neck_visual.stl
- link right_ankle: geometry collision box size=0.0656882356852293 0.094087990000844 0.05529999919235706; visual mesh filename=right_ankle_visual.stl
- link right_camera: mass 0 -> 1.01635e-23; geometry collision box size=9.999999747378752e-06 1.0163475963054225e-05 9.999999747378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; visual mesh filename=right_camera_visual.stl
- link right_foot: geometry collision box size=0.056986574083566666 0.13157938420772552 0.21582114696502686; visual mesh filename=right_foot_visual.stl
- link right_foot_base: mass 0 -> 1.01635e-23; geometry collision box size=9.999999747378752e-06 1.0163475963054225e-05 9.999999747378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; visual mesh filename=right_foot_base_visual.stl
- link right_hip_roll: geometry collision box size=0.06627646926790476 0.05529999919235706 0.09410000033676624; visual mesh filename=right_hip_roll_visual.stl
- link right_hip_yaw: geometry collision box size=0.10850000381469727 0.09402551129460335 0.07350000609436158; visual mesh filename=right_hip_yaw_visual.stl
- link right_lower_arm: geometry collision box size=0.08257202059030533 0.2583179399371147 0.05095679499208927; visual mesh filename=right_lower_arm_visual.stl
- link right_lower_leg: geometry collision box size=0.22920288890600204 0.03099999949336052 0.07800000160932541; visual mesh filename=right_lower_leg_visual.stl
- link right_shoulder: geometry collision box size=0.07999999821186066 0.08146718889474869 0.07936178296804419; visual mesh filename=right_shoulder_visual.stl
- link right_upper_arm: mass 0.134208 -> 0.299218; geometry collision box size=0.22480963170528412 0.079021405428648 0.08959505334496498; visual mesh filename=right_upper_arm_visual.stl
- link right_upper_leg: mass 0.136613 -> 0.313809; geometry collision box size=0.2462693639099598 0.09347053803503513 0.07300000265240669; visual mesh filename=right_upper_leg_visual.stl
- link torso: geometry collision box size=0.13950913399457932 0.1899828165769577 0.262624004855752; visual mesh filename=torso_visual.stl
Joints:
- removed joint left_knee
- removed joint neck_pitch
- removed joint right_knee
- added joint head_pitch: type revolute, parent neck, child head, origin xyz=-0.00024471 -0.000255294 0.0481 rpy=-1.5708 1.5708 0, axis 0 0 1, limit lower=-3.14159 upper=3.14159 effort=1 velocity=20
- added joint left_knee_pitch: type revolute, parent left_upper_leg, child left_lower_leg, origin xyz=0.206046 0.0569501 -1.44745e-14 rpy=-4.42146e-14 -3.94129e-15 -1.40554e-13, axis 0 0 1, limit lower=-3.14159 upper=3.14159 effort=1 velocity=20
- added joint right_knee_pitch: type revolute, parent right_upper_leg, child right_lower_leg, origin xyz=0.206046 0.0569501 -7.16788e-15 rpy=-7.0209e-15 3.9968e-14 -5.66214e-15, axis 0 0 1, limit lower=-3.14159 upper=3.14159 effort=1 velocity=20
- joint left_elbow_pitch: origin xyz=0.1575 -5.57465e-05 0.02695 rpy=1.5708 1.5708 0 -> xyz=0.1575 -5.57465e-05 0.02695 rpy=-1.5708 1.5708 0
- joint left_shoulder_pitch: origin xyz=-5.659e-18 0.077 0.17725 rpy=1.5708 1.5708 0 -> xyz=-5.659e-18 0.077 0.17725 rpy=-1.5708 1.5708 0
- joint left_shoulder_roll: origin xyz=0 0.0100012 -0.0479124 rpy=-1.5708 -3.06087e-14 1.5708 -> xyz=0 -0.0100012 0.0479124 rpy=1.5708 3.06087e-14 -1.5708
- joint right_elbow_pitch: origin xyz=0.1575 5.57465e-05 0.02695 rpy=1.5708 1.5708 0 -> xyz=0.1575 5.57465e-05 0.02695 rpy=-1.5708 1.5708 0
- joint right_shoulder_pitch: origin xyz=-3.55526e-17 -0.077 0.17725 rpy=1.5708 1.5708 0 -> xyz=-3.55526e-17 -0.077 0.17725 rpy=-1.5708 1.5708 0
- joint right_shoulder_roll: origin xyz=0 0.0100012 0.0479124 rpy=-1.5708 4.32987e-15 1.5708 -> xyz=0 -0.0100012 -0.0479124 rpy=1.5708 -4.32987e-15 -1.5708

Commit message: Revert pitch direction change

File: module/actuation/Kinematics/data/nugus.urdf (robot description, URDF)
Before this commit: robot onshape, 25 links, 24 joints
Links:
- link head: geometry collision box size=0.16223767679184675 0.15564338862895966 0.15779687464237213; visual mesh filename=head_visual.stl
- link left_lower_arm: geometry collision box size=0.08257202059030533 0.25829844921827316 0.050921617075800896; visual mesh filename=left_lower_arm_visual.stl
- link right_lower_arm: geometry collision box size=0.08257202059030533 0.2583179399371147 0.050956809893250465; visual mesh filename=right_lower_arm_visual.stl
- link right_upper_arm: geometry collision box size=0.22482992708683014 0.07902275025844574 0.08959516510367393; visual mesh filename=right_upper_arm_visual.stl
- link torso: geometry collision box size=0.13950913399457932 0.1899828165769577 0.2618043217808008; visual mesh filename=torso_visual.stl
Joints:
- joint head_pitch: origin xyz=-0.00024471 -0.000255294 0.0481 rpy=-1.5708 1.5708 0 -> xyz=-0.00024471 -0.000255294 0.0481 rpy=1.5708 1.5708 0
- joint left_camera: origin xyz=-0.0648803 0.0699522 -0.033795 rpy=-1.5708 1.63801e-13 1.53589 -> xyz=-0.0648803 -0.0699522 0.033795 rpy=1.5708 -1.63801e-13 -1.53589
- joint right_camera: origin xyz=-0.0648803 0.0699522 0.034205 rpy=-1.5708 1.63801e-13 1.53589 -> xyz=-0.0648803 -0.0699522 -0.034205 rpy=1.5708 -1.63801e-13 -1.53589

Commit message: Update nugus.urdf

File: module/actuation/Kinematics/data/nugus.urdf (robot description, URDF)
Before this commit: robot onshape, 25 links, 24 joints
Joints:
- joint left_foot_base: origin xyz=0.0360247 0 6.93889e-18 rpy=-1.71429e-29 -1.5708 0 -> xyz=0.038 6.93889e-18 1.38778e-17 rpy=-4.52109e-30 -1.5708 0
- joint right_foot_base: origin xyz=0.0360247 -1.38778e-17 0 rpy=-7.57306e-29 -1.5708 0 -> xyz=0.038 0 6.93889e-18 rpy=-1.26218e-29 -1.5708 0
