Commit message: Move to asset

File: nusight2/src/assets/nugus/robot.urdf (robot description, URDF)
Before this commit: robot onshape, 25 links, 24 joints
Links:
- link head: geometry collision box size=0.16223767679184675 0.15564338862895966 0.15779687464237213; visual mesh filename=./head_visual.stl
- link left_ankle: geometry collision box size=0.06627646926790476 0.09438799507915974 0.05529999919235706; visual mesh filename=./left_ankle_visual.stl
- link left_camera: geometry collision box size=9.999999747378752e-06 1.0163475963054225e-05 9.999999747323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; visual mesh filename=./left_camera_visual.stl
- link left_foot: geometry collision box size=0.05699313431978226 0.13158147037029266 0.21582108736038208; visual mesh filename=./left_foot_visual.stl
- link left_foot_base: geometry collision box size=9.999999747378752e-06 1.0163475963054225e-05 9.999999747378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; visual mesh filename=./left_foot_base_visual.stl
- link left_hip_roll: geometry collision box size=0.07245294097810984 0.05529999919235706 0.09385000355541706; visual mesh filename=./left_hip_roll_visual.stl
- link left_hip_yaw: geometry collision box size=0.10850000381469727 0.09402551129460335 0.07350000609436158; visual mesh filename=./left_hip_yaw_visual.stl
- link left_lower_arm: geometry collision box size=0.08257202059030533 0.25829844921827316 0.050921617075800896; visual mesh filename=./left_lower_arm_visual.stl
- link left_lower_leg: geometry collision box size=0.2292028944939375 0.03099999949336052 0.07800000160932541; visual mesh filename=./left_lower_leg_visual.stl
- link left_shoulder: geometry collision box size=0.07999999821186066 0.08144209161400795 0.0793731525540351; visual mesh filename=./left_shoulder_visual.stl
- link left_upper_arm: geometry collision box size=0.22483809292316437 0.07902275025844574 0.08959516510367393; visual mesh filename=./left_upper_arm_visual.stl
- link left_upper_leg: geometry collision box size=0.2462693639099598 0.09347053803503513 0.0729999989271164; visual mesh filename=./left_upper_leg_visual.stl
- link neck: geometry collision box size=0.04019999876618385 0.05000000074505806 0.062835298711434; visual mesh filename=./neck_visual.stl
- link right_ankle: geometry collision box size=0.0656882356852293 0.094087990000844 0.05529999919235706; visual mesh filename=./right_ankle_visual.stl
- link right_camera: geometry collision box size=9.999999747378752e-06 1.0163475963054225e-05 9.999999747378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; visual mesh filename=./right_camera_visual.stl
- link right_foot: geometry collision box size=0.056986574083566666 0.13157938420772552 0.21582114696502686; visual mesh filename=./right_foot_visual.stl
- link right_foot_base: geometry collision box size=9.999999747378752e-06 1.0163475963054225e-05 9.999999747378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; visual mesh filename=./right_foot_base_visual.stl
- link right_hip_roll: geometry collision box size=0.06627646926790476 0.05529999919235706 0.09410000033676624; visual mesh filename=./right_hip_roll_visual.stl
- link right_hip_yaw: geometry collision box size=0.10850000381469727 0.09402551129460335 0.07350000609436158; visual mesh filename=./right_hip_yaw_visual.stl
- link right_lower_arm: geometry collision box size=0.08257202059030533 0.2583179399371147 0.050956809893250465; visual mesh filename=./right_lower_arm_visual.stl
- link right_lower_leg: geometry collision box size=0.22920288890600204 0.03099999949336052 0.07800000160932541; visual mesh filename=./right_lower_leg_visual.stl
- link right_shoulder: geometry collision box size=0.07999999821186066 0.08146718889474869 0.07936178296804419; visual mesh filename=./right_shoulder_visual.stl
- link right_upper_arm: geometry collision box size=0.22482992708683014 0.07902275025844574 0.08959516510367393; visual mesh filename=./right_upper_arm_visual.stl
- link right_upper_leg: geometry collision box size=0.2462693639099598 0.09347053803503513 0.07300000265240669; visual mesh filename=./right_upper_leg_visual.stl
- link torso: geometry collision box size=0.13950913399457932 0.1899828165769577 0.2618043217808008; visual mesh filename=./torso_visual.stl

Commit message: Fix right_ankle_pitch limits

File: nusight2/src/assets/nugus/robot.urdf (robot description, URDF)
Before this commit: robot onshape, 25 links, 24 joints
Links:
- link head: geometry collision box size=0.16223767679184675 0.15564338862895966 0.15779687464237213; visual mesh filename=head_visual.stl
- link left_ankle: geometry collision box size=0.06568823475390673 0.09438799507915974 0.05529999919235706; visual mesh filename=left_ankle_visual.stl
- link left_camera: geometry collision box size=9.999999747378752e-06 1.0163475963054225e-05 9.999999747323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; visual mesh filename=left_camera_visual.stl
- link left_foot: geometry collision box size=0.05699313431978226 0.13158147037029266 0.21582108736038208; visual mesh filename=left_foot_visual.stl
- link left_foot_base: geometry collision box size=9.999999747378752e-06 1.0163475963054225e-05 9.999999747378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; visual mesh filename=left_foot_base_visual.stl
- link left_hip_roll: geometry collision box size=0.07245294097810984 0.05529999919235706 0.09385000355541706; visual mesh filename=left_hip_roll_visual.stl
- link left_hip_yaw: geometry collision box size=0.10850000381469727 0.09402551129460335 0.07350000609436158; visual mesh filename=left_hip_yaw_visual.stl
- link left_lower_arm: geometry collision box size=0.08257202059030533 0.25829844921827316 0.050921617075800896; visual mesh filename=left_lower_arm_visual.stl
- link left_lower_leg: geometry collision box size=0.2292028944939375 0.03099999949336052 0.07800000160932541; visual mesh filename=left_lower_leg_visual.stl
- link left_shoulder: geometry collision box size=0.07999999821186066 0.08144209161400795 0.0793731525540351; visual mesh filename=left_shoulder_visual.stl
- link left_upper_arm: geometry collision box size=0.22483809292316437 0.07902275025844574 0.08959516510367393; visual mesh filename=left_upper_arm_visual.stl
- link left_upper_leg: geometry collision box size=0.2462693639099598 0.09347053803503513 0.0729999989271164; visual mesh filename=left_upper_leg_visual.stl
- link neck: geometry collision box size=0.04019999876618385 0.05000000074505806 0.062835298711434; visual mesh filename=neck_visual.stl
- link right_ankle: geometry collision box size=0.0656882356852293 0.094087990000844 0.05529999919235706; visual mesh filename=right_ankle_visual.stl
- link right_camera: geometry collision box size=9.999999747378752e-06 1.0163475963054225e-05 9.999999747378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; visual mesh filename=right_camera_visual.stl
- link right_foot: geometry collision box size=0.056986574083566666 0.13157938420772552 0.21582114696502686; visual mesh filename=right_foot_visual.stl
- link right_foot_base: geometry collision box size=9.999999747378752e-06 1.0163475963054225e-05 9.999999747378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; visual mesh filename=right_foot_base_visual.stl
- link right_hip_roll: geometry collision box size=0.06627646926790476 0.05529999919235706 0.09410000033676624; visual mesh filename=right_hip_roll_visual.stl
- link right_hip_yaw: geometry collision box size=0.10850000381469727 0.09402551129460335 0.07350000609436158; visual mesh filename=right_hip_yaw_visual.stl
- link right_lower_arm: geometry collision box size=0.08257202059030533 0.2583179399371147 0.050956809893250465; visual mesh filename=right_lower_arm_visual.stl
- link right_lower_leg: geometry collision box size=0.22920288890600204 0.03099999949336052 0.07800000160932541; visual mesh filename=right_lower_leg_visual.stl
- link right_shoulder: geometry collision box size=0.07999999821186066 0.08146718889474869 0.07936178296804419; visual mesh filename=right_shoulder_visual.stl
- link right_upper_arm: geometry collision box size=0.22482992708683014 0.07902275025844574 0.08959516510367393; visual mesh filename=right_upper_arm_visual.stl
- link right_upper_leg: geometry collision box size=0.2462693639099598 0.09347053803503513 0.07300000265240669; visual mesh filename=right_upper_leg_visual.stl
- link torso: geometry collision box size=0.13950913399457932 0.1899828165769577 0.2618043217808008; visual mesh filename=torso_visual.stl
Joints:
- joint left_ankle_pitch: origin xyz=0.200203 -3.46945e-17 6.93889e-18 rpy=-3.05311e-15 5.55112e-17 -2.87748e-14 -> xyz=0.200203 -3.46945e-17 0 rpy=-9.74385e-15 5.86234e-16 -1.54846e-15
- joint left_ankle_roll: origin xyz=0 0 6.93889e-18 rpy=1.5708 3.37316e-16 -3.88578e-16 -> xyz=0 -1.38778e-17 -2.08167e-17 rpy=1.5708 6.70375e-15 -2.75955e-14
- joint left_foot_base: origin xyz=0.038 6.93889e-18 1.38778e-17 rpy=-4.52109e-30 -1.5708 0 -> xyz=0.038 0 0 rpy=-2.39955e-29 -1.5708 0
- joint left_hip_pitch: origin xyz=0 -6.93889e-18 -1.38778e-17 rpy=-1.5708 -1.29896e-14 3.34849e-14 -> xyz=1.38778e-17 0 -1.04083e-17 rpy=-1.5708 -1.78655e-11 3.29833e-14
- joint left_hip_roll: origin xyz=0.0221332 0 -0.0545 rpy=-4.55628e-30 1.5708 0 -> xyz=0.0221332 2.91434e-16 -0.0545 rpy=6.66729e-21 1.5708 0
- joint left_knee_pitch: origin xyz=0.206046 0.0569501 -1.44745e-14 rpy=-4.42146e-14 -3.94129e-15 -1.40554e-13 -> xyz=0.206046 0.0569501 -1.44676e-14 rpy=-3.82657e-14 -3.77567e-15 0.00480121
- joint right_ankle_pitch: limit effort=1 velocity=20 -> lower=-3.14159 upper=3.14159 effort=1 velocity=20
