Commit message: Invert head pitch direction

File: shared/utility/platform/models/nugus.urdf (robot description, URDF)
Before this commit: robot onshape, 25 links, 24 joints
Joints:
- joint head_pitch: origin xyz=-0.00024471 -0.000255294 0.0481 rpy=1.5708 1.5708 0 -> xyz=-0.00024471 -0.000255294 0.0481 rpy=-1.5708 1.5708 0
- joint left_camera: origin xyz=-0.0648803 -0.0699522 0.033795 rpy=1.5708 -1.63801e-13 -1.53589 -> xyz=-0.0648803 0.0699522 -0.033795 rpy=-1.5708 1.63801e-13 1.53589
- joint right_camera: origin xyz=-0.0648803 -0.0699522 -0.034205 rpy=1.5708 -1.63801e-13 -1.53589 -> xyz=-0.0648803 0.0699522 0.034205 rpy=-1.5708 1.63801e-13 1.53589

Commit message: Revert "Invert head pitch direction"
This reverts commit 43784dfb2098a2a948a8374e81c021120d3d5c5d.

File: shared/utility/platform/models/nugus.urdf (robot description, URDF)
Before this commit: robot onshape, 25 links, 24 joints
Joints:
- joint head_pitch: origin xyz=-0.00024471 -0.000255294 0.0481 rpy=-1.5708 1.5708 0 -> xyz=-0.00024471 -0.000255294 0.0481 rpy=1.5708 1.5708 0
- joint left_camera: origin xyz=-0.0648803 0.0699522 -0.033795 rpy=-1.5708 1.63801e-13 1.53589 -> xyz=-0.0648803 -0.0699522 0.033795 rpy=1.5708 -1.63801e-13 -1.53589
- joint right_camera: origin xyz=-0.0648803 0.0699522 0.034205 rpy=-1.5708 1.63801e-13 1.53589 -> xyz=-0.0648803 -0.0699522 -0.034205 rpy=1.5708 -1.63801e-13 -1.53589

Commit message: Update nugus.urdf

File: shared/utility/platform/models/nugus.urdf (robot description, URDF)
Before this commit: robot onshape, 25 links, 24 joints
Links:
- link left_ankle: geometry collision box size=0.06568823475390673 0.09438799507915974 0.05529999919235706; visual mesh filename=left_ankle_visual.stl
Joints:
- joint left_ankle_pitch: origin xyz=0.200203 -3.46945e-17 6.93889e-18 rpy=-3.05311e-15 5.55112e-17 -2.87748e-14 -> xyz=0.200203 -3.46945e-17 0 rpy=-9.74385e-15 5.86234e-16 -1.54846e-15
- joint left_ankle_roll: origin xyz=0 0 6.93889e-18 rpy=1.5708 3.37316e-16 -3.88578e-16 -> xyz=0 -1.38778e-17 -2.08167e-17 rpy=1.5708 6.70375e-15 -2.75955e-14
- joint left_foot_base: origin xyz=0.038 6.93889e-18 1.38778e-17 rpy=-4.52109e-30 -1.5708 0 -> xyz=0.038 0 0 rpy=-2.39955e-29 -1.5708 0
- joint left_hip_pitch: origin xyz=0 -6.93889e-18 -1.38778e-17 rpy=-1.5708 -1.29896e-14 3.34849e-14 -> xyz=1.38778e-17 0 -1.04083e-17 rpy=-1.5708 -1.78655e-11 3.29833e-14
- joint left_hip_roll: origin xyz=0.0221332 0 -0.0545 rpy=-4.55628e-30 1.5708 0 -> xyz=0.0221332 2.91434e-16 -0.0545 rpy=6.66729e-21 1.5708 0
- joint left_knee_pitch: origin xyz=0.206046 0.0569501 -1.44745e-14 rpy=-4.42146e-14 -3.94129e-15 -1.40554e-13 -> xyz=0.206046 0.0569501 -1.44676e-14 rpy=-3.82657e-14 -3.77567e-15 0.00480121
- joint right_ankle_pitch: limit effort=1 velocity=20 -> lower=-3.14159 upper=3.14159 effort=1 velocity=20
