Commit message: Rename head_yaw and head_pitch to be more consistent

File: shared/utility/platform/models/nugus/robot.urdf (robot description, URDF)
Before this commit: robot onshape, 25 links, 24 joints
Joints:
- removed joint neck_yaw
- added joint head_yaw: type revolute, parent torso, child neck, origin xyz=-0.008 2.09034e-16 0.20825 rpy=-1.1045e-15 2.10942e-15 -3.14159, axis 0 0 1, limit lower=-3.14159 upper=3.14159 effort=1 velocity=20

Commit message: change head_yaw to neck_yaw to match NUWebots usage

File: shared/utility/platform/models/nugus/robot.urdf (robot description, URDF)
Before this commit: robot onshape, 25 links, 24 joints
Joints:
- removed joint head_yaw
- added joint neck_yaw: type revolute, parent torso, child neck, origin xyz=-0.008 2.09034e-16 0.20825 rpy=-1.1045e-15 2.10942e-15 -3.14159, axis 0 0 1, limit lower=-3.14159 upper=3.14159 effort=1 velocity=20
