Commit message: Tune extrinsics

File: nusight2/src/assets/robot-models/k1/robot.urdf (robot description, URDF)
Before this commit: robot K1, 23 links, 22 joints
Links:
- added link camera_link, mass 0.001
Joints:
- added joint camera: type fixed, parent Head_2, child camera_link, origin xyz=-0.0122268423 0.0440084077 -0.0283811111 rpy=-1.5518693404 -0.0017597899 -1.4953884566

Commit message: Tidy up and remove tinyrobotics dep

File: nusight2/src/assets/robot-models/k1/robot.urdf (robot description, URDF)
Before this commit: robot K1, 24 links, 23 joints
Links:
- removed link camera_link
Joints:
- removed joint camera
